File: hardware/Prototype/Prototype.kicad_pcb (KiCad board)
At the start: 2 copper layers, 83.8 x 68.6 mm, 11 parts, among them J1 Conn_01x16_Socket, J2 Conn_01x12_Socket, J3 Conn_01x03_Socket, J4 Conn_01x03_Socket, J5 Conn_01x02_Socket, J6 Conn_01x04_Socket, J7 Conn_01x02_Socket, J8 Conn_01x02_Socket

Commit message: Finished schematics for presentation
Other:
- board text added: "9V Battery"
Changed lines of the file:
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@@
 		(tags "Through hole socket strip THT 1x03 2.54mm single row")
 		(property "Reference" "J4"
-			(at 0 -2.77 270)
+			(at 0 -2.77 -90)
 			(layer "F.SilkS")
 			(effects
@@
 		)
 		(property "Value" "Conn_01x03_Socket"
-			(at 0 7.85 270)
+			(at 0 7.85 -90)
 			(layer "F.Fab")
 			(effects
@@
 		)
 		(fp_text user "${REFERENCE}"
-			(at 0 2.54 360)
+			(at 0 2.54 0)
 			(layer "F.Fab")
 			(effects
@@
 		(tags "Resistor Axial_DIN0207 series Axial Horizontal pin pitch 10.16mm 0.25W = 1/4W length 6.3mm diameter 2.5mm")
 		(property "Reference" "R1"
-			(at 5.08 -2.37 360)
+			(at 5.08 -2.37 0)
 			(layer "F.SilkS")
 			(effects
@@
 		)
 		(property "Value" "220R"
-			(at 5.08 2.37 360)
+			(at 5.08 2.37 0)
 			(layer "F.Fab")
 			(effects
@@
 		)
 		(fp_text user "${REFERENCE}"
-			(at 5.08 0 360)
+			(at 5.08 0 0)
 			(layer "F.Fab")
 			(effects
@@
 		(tags "C Axial series Axial Horizontal pin pitch 10mm  length 5.1mm diameter 3.1mm")
 		(property "Reference" "C1"
-			(at 5 -2.67 360)
+			(at 5 -2.67 0)
 			(layer "F.SilkS")
 			(effects
@@
 		)
 		(property "Value" "100n"
-			(at 5 2.67 360)
+			(at 5 2.67 0)
 			(layer "F.Fab")
 			(effects
@@
 		)
 		(fp_text user "${REFERENCE}"
-			(at 5 0 360)
+			(at 5 0 0)
 			(layer "F.Fab")
 			(effects
@@
 		(tags "Through hole socket strip THT 1x02 2.54mm single row")
 		(property "Reference" "J8"
-			(at 0 -2.77 270)
+			(at 0 -2.77 -90)
 			(layer "F.SilkS")
 			(effects
@@
 		)
 		(property "Value" "Conn_01x02_Socket"
-			(at 0 5.31 270)
+			(at 0 5.31 -90)
 			(layer "F.Fab")
 			(effects
@@
 		)
 		(fp_text user "${REFERENCE}"
-			(at 0 1.27 360)
+			(at 0 1.27 0)
 			(layer "F.Fab")
 			(effects
@@
 		(layer "Edge.Cuts")
 	)
+	(gr_text "9V Battery"
+		(at 124.46 85.92 0)
+		(layer "F.SilkS")
+		(effects
+			(font
+				(size 4 4)
+				(thickness 0.75)
+			)
+			(justify left bottom)
+		)
+	)
 	(segment
