File: hardware/Prototype/Prototype.kicad_sch (KiCad schematic)
At the start: 11 parts, among them J1 Conn_01x16_Socket, J2 Conn_01x12_Socket, J3 Conn_01x03_Socket, J4 Conn_01x03_Socket, J5 Conn_01x02_Socket, J6 Conn_01x04_Socket, J7 Conn_01x02_Socket, J8 Conn_01x02_Socket

Commit message: Misc
Parts:
- added OP1, OP101, OP2, OP3: ${SIM.PARAMS}, symbol Simulation_SPICE:OPAMP
- added PTC1: 100R @ 0 deg C, symbol Device:Thermistor_PTC
- added R1, R103: 100R, Resistor_THT:R_Axial_DIN0207_L6.3mm_D2.5mm_P10.16mm_Horizontal, symbol Device:R
- added R101: 2k2, Resistor_THT:R_Axial_DIN0207_L6.3mm_D2.5mm_P10.16mm_Horizontal, symbol Device:R
- added R102: 1k, Resistor_THT:R_Axial_DIN0207_L6.3mm_D2.5mm_P10.16mm_Horizontal, symbol Device:R
- added R2, R3: 110R, Resistor_THT:R_Axial_DIN0207_L6.3mm_D2.5mm_P10.16mm_Horizontal, symbol Device:R
- R1: value 220R -> 100R
Connections:
- net +3V3: now also OP1.3 (V+), OP101.3 (V+), OP2.3 (V+), OP3.3 (V+), PTC1.1, R1.2
- net GND: now also OP1.4 (V-), OP101.4 (V-), OP2.4 (V-), OP3.4 (V-), R102.1, R2.1, R3.1
- net PT_OUT: now also OP101.5, R103.1
- net BAT_SENSE: now reaches J1.6 (Pin_6)
- net BAT_SENSE: now also R101.1, R102.2
- net +BATT renamed +BAT
- net +BAT: now also R101.2
- new net: OP2.1 (+), PTC1.2, R3.2
- new net: OP1.1 (+), R1.1, R2.2
- new net: OP1.2 (-), OP1.5, OP3.1 (+)
- new net: OP2.2 (-), OP2.5, OP3.2 (-)
- no-connect marks 19 -> 18
Other:
- note added: "R101 and R102 chosen for +BAT <= 10.5V"
- company: (none) -> Alfred Wrigfors
- title: (none) -> Applied IoT
- moved on the sheet: C1, D1, J1, J2, J3, J4, J5, J6, J7, J8, R1

Commit message: Finished schematics for presentation
Parts:
- removed OP1, OP101, OP2, OP3: ${SIM.PARAMS}, symbol Simulation_SPICE:OPAMP
- removed PTC1: 100R @ 0 deg C, symbol Device:Thermistor_PTC
- removed R1, R103: 100R, Resistor_THT:R_Axial_DIN0207_L6.3mm_D2.5mm_P10.16mm_Horizontal, symbol Device:R
- removed R2, R3: 110R, Resistor_THT:R_Axial_DIN0207_L6.3mm_D2.5mm_P10.16mm_Horizontal, symbol Device:R
